File: MINI VESC.kicad_sch (KiCad schematic)
At the start: 151 parts, among them P1 CONN_1, P10 CONN_01X06, P11 CONN_01X06, P2 CONN_1, P3 CONN_1, P4 CONN_1, P5 CONN_1, P6 CONN_1, P9 CONN_01X06, Q1 NTMFS5C604NLT1G, Q2 NTMFS5C604NLT1G, Q3 NTMFS5C604NLT1G, Q4 NTMFS5C604NLT1G, Q5 NTMFS5C604NLT1G, Q6 NTMFS5C604NLT1G, U1 LM5113SDE, U10 MCP1700, U2 LM5113SDE, U3 LM5113SDE, U4 AD8417, U5 AD8417, U6 AD8417, U7 STM32F405RGT6, U8 LMR16006YDDCT, U9 MCP1700, X1 ABM3B-8.000MHZ

Commit message: Lots of stuff
Parts:
- removed C1, C2, C3: 470n, Capacitors_SMD:C_0603, symbol Device:C
- removed C10, C11, C6, C7, C8, C9: 2u2, Capacitors_SMD:C_0603, symbol Device:C
- removed C12, C13, C28, C32, C39, C4, C48, C5, C60, C61, C62, C63, C74, C75, C79, C80, C82, C84, C85: 10u, Resistors_SMD:R_1206, symbol Device:C
- removed C33, C34, C35, C36, C37, C38, C40, C41, C42, C43, C44, C45, C46, C47, C49, C50, C51, C52, C53, C54, C55, C56, C57, C58, C59, C64, C65, C66, C67, C68, C69, C70, C71, C72, C73, C81, C83: C, Resistors_SMD:R_1206, symbol Device:C
- removed P1, P2, P3, P4, P5, P6: CONN_1, kicad_subory:prekov, symbol MINI VESC-rescue:CONN_1-RESCUE-MINI_VESC
- removed Q1, Q2, Q3, Q4, Q5, Q6: NTMFS5C604NLT1G, kicad_subory:DFN5, symbol Device:Q_NMOS_GSD
- removed R1, R2, R3: R0005, mojaKniznica:2512Rv2, symbol MINI VESC-rescue:RSENS-RESCUE-MINI_VESC
- removed R10, R11, R6, R7, R8, R9: 3R9, Resistors_SMD:R_0603, symbol Device:R
- removed R12, R14: 39k, Resistors_SMD:R_0603, symbol Device:R
- removed R13, R15, R17: 2k2, Resistors_SMD:R_0603, symbol Device:R
- removed R16: 25k5, Resistors_SMD:R_0603, symbol Device:R
- removed U1, U2, U3: LM5113SDE, kicad_subory:WSON10__, symbol MINI VESC-rescue:LM5001-RESCUE-MINI_VESC
- removed U4, U5, U6: AD8417, kicad_subory:MSOP, symbol MINI VESC-rescue:AD8418-RESCUE-MINI_VESC
- C14, C15, C16, C17, C18, C19, C20, C21, C22, C26, C27, C29, C30, C31, C77, C78, C86, C87, C88, C89, C90: footprint Capacitors_SMD:C_0603 -> Capacitor_SMD:C_0603_1608Metric
- C23, C76: footprint Resistors_SMD:R_0603 -> Capacitor_SMD:C_0603_1608Metric
- C24, C25: footprint Resistors_SMD:R_1206 -> Capacitor_SMD:C_1206_3216Metric
- D3, D4: footprint Resistors_SMD:R_0603 -> LED_SMD:LED_0603_1608Metric
- R18, R19, R20, R21, R22, R25, R27, R28, R29, R30, R31, R32, R33, R34, R4, R5: footprint Resistors_SMD:R_0603 -> Resistor_SMD:R_0603_1608Metric
Other:
- added sheet Capacitor Bank (capacitor-bank.kicad_sch)
- added sheet Half Bridge U (half-bridge.kicad_sch)
- added sheet Half Bridge V (half-bridge.kicad_sch)
- added sheet Half Bridge W (half-bridge.kicad_sch)
- note removed: "56x 2u2 100V"

Commit message: More work
Parts:
- removed C14, C15, C16: 4n7, Capacitor_SMD:C_0603_1608Metric, symbol Device:C
- removed R18, R19, R20: 100R, Resistor_SMD:R_0603_1608Metric, symbol Device:R
Connections:
- net LI1: no longer U7.34 (PB13(OTG_HS_VBUS))
- net TEMP_MOTOR: no longer P9.2 (Pin_2), U7.24 (PC4(ADC12_IN14))
- net C1 renamed I_{senseU}
- net C2 renamed I_{senseV}
- net C3 renamed I_{senseW}
- net SENS_1 renamed V_{senseU}
- net SENS_2 renamed V_{senseV}
- net SENS_3 renamed V_{senseW}
- net SENS_SUPPLY renamed Supply_{sense}
- new net Switch_{lowU}: U7.34 (PB13(OTG_HS_VBUS))
- new net T_{motor}: P9.2 (Pin_2), U7.24 (PC4(ADC12_IN14))
Other:
- moved on the sheet: D3, D4, R28, R29
