File: psu.kicad_sch (KiCad schematic)
At the start: 3 parts, among them U1 MCP1700x-330xxTT

Commit message: Playing around with routing
Parts:
- renumbered C15 to C87, C16 to C88, U1 to U9
Changed lines of the file:
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@@
   (symbol (lib_id "Device:C") (at 38.1 46.99 0) (unit 1)
     (in_bom yes) (on_board yes) (dnp no)
-    (property "Reference" "C15" (at 37.465 44.45 0)
+    (property "Reference" "C87" (at 37.465 44.45 0)
       (effects (font (size 1.27 1.27)) (justify right))
     )
@@
       (project "mini-vesc"
         (path "/994820bf-9e2d-4c1b-8cdf-e9baf8707794/bdbc759a-b717-4eff-99a0-9bf280e00dfc"
-          (reference "C15") (unit 1)
+          (reference "C87") (unit 1)
         )
         (path "/994820bf-9e2d-4c1b-8cdf-e9baf8707794/c70c1ef2-97a2-4249-b37b-9719b3c7377c"
-          (reference "C15") (unit 1)
+          (reference "C89") (unit 1)
         )
       )
@@
   (symbol (lib_id "Device:C") (at 74.93 46.99 0) (unit 1)
     (in_bom yes) (on_board yes) (dnp no)
-    (property "Reference" "C16" (at 74.295 44.45 0)
+    (property "Reference" "C88" (at 74.295 44.45 0)
       (effects (font (size 1.27 1.27)) (justify right))
     )
@@
       (project "mini-vesc"
         (path "/994820bf-9e2d-4c1b-8cdf-e9baf8707794/bdbc759a-b717-4eff-99a0-9bf280e00dfc"
-          (reference "C16") (unit 1)
+          (reference "C88") (unit 1)
         )
         (path "/994820bf-9e2d-4c1b-8cdf-e9baf8707794/c70c1ef2-97a2-4249-b37b-9719b3c7377c"
-          (reference "C16") (unit 1)
+          (reference "C90") (unit 1)
         )
       )
@@
   (symbol (lib_id "Regulator_Linear:MCP1700x-330xxTT") (at 55.88 38.1 0) (unit 1)
     (in_bom yes) (on_board yes) (dnp no)
-    (property "Reference" "U1" (at 52.07 34.925 0)
+    (property "Reference" "U9" (at 52.07 34.925 0)
       (effects (font (size 1.27 1.27)))
     )
@@
       (project "mini-vesc"
         (path "/994820bf-9e2d-4c1b-8cdf-e9baf8707794/bdbc759a-b717-4eff-99a0-9bf280e00dfc"
-          (reference "U1") (unit 1)
+          (reference "U9") (unit 1)
         )
         (path "/994820bf-9e2d-4c1b-8cdf-e9baf8707794/c70c1ef2-97a2-4249-b37b-9719b3c7377c"
-          (reference "U1") (unit 1)
+          (reference "U10") (unit 1)
         )
       )
