File: capacitor-bank.kicad_sch (KiCad schematic)
At the start: 56 parts

Commit message: Playing around with routing
Parts:
- renumbered C4 to C19, C66 to C20, C13 to C21, C5 to C22, C81 to C23, C85 to C24, C32 to C25, C33 to C26, C72 to C27, C36 to C28, C34 to C29, C12 to C30, C38 to C31, C49 to C32, C39 to C33, C83 to C34, C42 to C35, C40 to C36, C35 to C37, C44 to C38, C55 to C39, C45 to C40, C71 to C41, C48 to C42, C46 to C43, C41 to C44, C50 to C45, C61 to C46, C51 to C47, C82 to C48, C54 to C49, C52 to C50, C47 to C51, C56 to C52, C67 to C53, C57 to C54, C58 to C55, C60 to C56, C75 to C57, C53 to C58, C62 to C59, C73 to C60, C63 to C61, C64 to C62, C28 to C63, C79 to C64, C59 to C65, C68 to C66, C84 to C67, C69 to C68, C70 to C69, C37 to C70, C80 to C71, C65 to C72, C74 to C73, C43 to C74

Commit message: More work
Parts:
- C19, C22, C24, C29, C31, C32, C36, C39, C46, C48, C52, C53, C59, C60, C63, C66, C67, C70, C73: value 10u -> 2.2µF; Class (none) -> X7R; Voltage (none) -> 100V
- C20, C21, C23, C25, C26, C27, C28, C30, C33, C34, C35, C37, C38, C40, C41, C42, C43, C44, C45, C47, C49, C50, C51, C54, C55, C56, C57, C58, C61, C62, C64, C65, C68, C69, C71, C72, C74: value C -> 2.2µF; Class (none) -> X7R; Voltage (none) -> 100V
Other:
- note added: "56x 2.2µF, 100V"
- note removed: "56x 2u2 100V"
