File: mini-vesc.kicad_sch (KiCad schematic)
At the start: 47 parts, among them P10 CONN_01X06, P11 CONN_01X06, P9 CONN_01X06, U10 MCP1700, U7 STM32F405RGT6, U8 LMR16006YDDCT, U9 MCP1700, X1 ABM3B-8.000MHZ

Commit message: More work
Parts:
- U?: renamed from U9; value MCP1700 -> MCP1700x-330xxTT; footprint TO_SOT_Packages_SMD:SOT-23 -> Package_TO_SOT_SMD:SOT-23; symbol MINI VESC-rescue:MCP1700-RESCUE-MINI_VESC -> Regulator_Linear:MCP1700x-330xxTT
- U?: renamed from U10; value MCP1700 -> MCP1700x-330xxTT; footprint TO_SOT_Packages_SMD:SOT-23 -> Package_TO_SOT_SMD:SOT-23; symbol MINI VESC-rescue:MCP1700-RESCUE-MINI_VESC -> Regulator_Linear:MCP1700x-330xxTT
Other:
- sheet Half Bridge U ports: added Phase; removed none
- sheet Half Bridge V ports: added Phase; removed none
- sheet Half Bridge W ports: added Phase; removed none
- moved on the sheet: C87, C88, C89, C90, U?

Commit message: More work
Parts:
- removed C87, C88, C89, C90: 2u2, Capacitor_SMD:C_0603_1608Metric, symbol Device:C
- removed U? (x2): MCP1700x-330xxTT, Package_TO_SOT_SMD:SOT-23, symbol Regulator_Linear:MCP1700x-330xxTT
- C17, C18, C24, C77, C78, C86: value 2u2 -> 2.2µF
- C19, C21, C22, C26, C27, C29, C76: value 100n -> 100nF
- C25: value 10u -> 10µF
- R21, R31, R34: value 10k -> 10kΩ
- R22: value 54k9 -> 54.9kΩ
- R25, R27: value 22R -> 22Ω
- R28, R29: value 220R -> 220Ω
- R30: value 100R -> 100Ω
- R32: value 10kNTC -> 10kΩ; MPN (none) -> NCP18XH103F03RB; Manufacturer (none) -> Murata
- R33: value 100k -> 100kΩ
- R4: value 39k -> 39kΩ
- R5: value 2k2 -> 2.2kΩ
Other:
- added sheet PSU - Analog (psu.kicad_sch)
- added sheet PSU - Digital (psu.kicad_sch)
- moved on the sheet: C19, C21, C22, C26, C27, C29, C86, D3, D4, P11, R28, R29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

Commit message: Playing around with routing
Parts:
- renumbered C23 to C1, C77 to C10, C78 to C11, C30 to C12, C17 to C13, C18 to C14, C20 to C15, C19 to C16, C31 to C17, C86 to C18, C24 to C2, C76 to C3, C25 to C4, C29 to C5, C21 to C6, C22 to C7, C26 to C8, C27 to C9, D3 to D2, D4 to D3, P11 to P1, P10 to P2, P9 to P3, R21 to R1, R31 to R10, R32 to R11, R25 to R12, R27 to R13, R22 to R2, R33 to R3, R30 to R4, R4 to R5, R5 to R6, R29 to R7, R28 to R8, R34 to R9, U8 to U1, U7 to U2

Commit message: More work
Parts:
- C12, C17: Class (none) -> C0G
- C15: value 100n -> 100nF
- C2: Class (none) -> X7R; Voltage (none) -> 100V
Changed lines of the file:
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@@
       (effects (font (size 1.27 1.27)) (justify left))
     )
-    (property "Value" "100n" (at 284.48 46.99 0)
+    (property "Value" "100nF" (at 284.48 46.99 0)
       (effects (font (size 1.27 1.27)) (justify left))
     )
@@
       (effects (font (size 1.27 1.27)) hide)
     )
+    (property "Class" "X7R" (at 58.42 181.61 0)
+      (effects (font (size 1.27 1.27)) hide)
+    )
+    (property "Voltage" "100V" (at 58.42 181.61 0)
+      (effects (font (size 1.27 1.27)) hide)
+    )
     (pin "2")
     (pin "1")
@@
       (effects (font (size 1.27 1.27)) hide)
     )
+    (property "Class" "C0G" (at 267.97 21.59 0)
+      (effects (font (size 1.27 1.27)) hide)
+    )
     (pin "1")
     (pin "2")
@@
       (effects (font (size 1.27 1.27)) hide)
     )
+    (property "Class" "C0G" (at 280.67 21.59 0)
+      (effects (font (size 1.27 1.27)) hide)
+    )
