File: half-bridge.kicad_sch (KiCad schematic)
At the start: 14 parts, among them P1 CONN_1, P4 CONN_1, Q1 NTMFS5C604NLT1G, Q2 NTMFS5C604NLT1G, U1 LM5113SDE, U4 AD8417

Commit message: More work
Parts:
- added C2: 4.7nF, Capacitor_SMD:C_0603_1608Metric, symbol Device:C
- added R2: 100R, Resistor_SMD:R_0603_1608Metric, symbol Device:R
- U4: footprint kicad_subory:MSOP -> Package_SO:MSOP-8_3x3mm_P0.65mm
Connections:
- net I_{sense}: now also C2.2, R2.2; no longer U4.5 (OUT)
- net VSS: now also C2.1
- new net: R2.1, U4.5 (OUT)

Commit message: More work
Parts:
- added U2: ~, symbol Symbols:LM5113-Q1
Connections:
- net High: now also U2.6 (HI); no longer U1.7 (HI)
- net Low: now also U2.7 (LI); no longer U1.8 (LI)
Changed lines of the file:
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@@
-    (stroke (width 0) (type default))
-  )
-  (wire (pts (xy 91.44 68.58) (xy 99.06 68.58))
     (stroke (width 0) (type default))
   )
@@
     (stroke (width 0) (type default))
   )
+  (wire (pts (xy 92.71 115.57) (xy 100.33 115.57))
+    (stroke (width 0) (type default))
+  )
   (wire (pts (xy 198.12 100.33) (xy 198.12 102.87))
     (stroke (width 0) (type default))
@@
     (stroke (width 0) (type default))
   )
+  (wire (pts (xy 92.71 110.49) (xy 100.33 110.49))
+    (stroke (width 0) (type default))
+  )
   (wire (pts (xy 245.11 96.52) (xy 242.57 96.52))
     (stroke (width 0) (type default))
@@
   )
   (wire (pts (xy 198.12 77.47) (xy 226.06 77.47))
-    (stroke (width 0) (type default))
-  )
-  (wire (pts (xy 91.44 63.5) (xy 99.06 63.5))
     (stroke (width 0) (type default))
   )
@@
     (effects (font (size 1.524 1.524)) (justify left))
   )
-  (hierarchical_label "Low" (shape input) (at 91.44 68.58 180) (fields_autoplaced)
+  (hierarchical_label "Low" (shape input) (at 92.71 115.57 180) (fields_autoplaced)
+    (effects (font (size 1.524 1.524)) (justify right))
+  )
+  (hierarchical_label "High" (shape input) (at 92.71 110.49 180) (fields_autoplaced)
     (effects (font (size 1.524 1.524)) (justify right))
   )
   (hierarchical_label "I_{sense}" (shape input) (at 265.43 93.98 0) (fields_autoplaced)
     (effects (font (size 1.524 1.524)) (justify left))
-  )
-  (hierarchical_label "High" (shape input) (at 91.44 63.5 180) (fields_autoplaced)
-    (effects (font (size 1.524 1.524)) (justify right))
   )
   (symbol (lib_id "Device:R") (at 252.73 93.98 90) (unit 1)
@@
         )
       )
+    )
+  )
+  (symbol (lib_id "Symbols:LM5113-Q1") (at 110.49 113.03 0) (unit 1)
+    (in_bom yes) (on_board yes) (dnp no) (fields_autoplaced)
+    (property "Reference" "U2" (at 112.6841 97.79 0)
+      (effects (font (size 1.27 1.27)) (justify left))
+    )
+    (property "Value" "~" (at 110.49 111.76 0)
+      (effects (font (size 1.27 1.27)))
+    )
+    (property "Footprint" "" (at 110.49 111.76 0)
+      (effects (font (size 1.27 1.27)) hide)
+    )
+    (property "Datasheet" "" (at 110.49 111.76 0)
+      (effects (font (size 1.27 1.27)) hide)
+    )
+    (pin "8")
+    (pin "7")
+    (pin "6")
+    (pin "4")
+    (pin "9")
+    (pin "5")
+    (pin "3")
+    (pin "2")
+    (pin "11")
+    (pin "1")
+    (pin "10")
+    (instances
+      (project "MINI VESC"
+        (path "/994820bf-9e2d-4c1b-8cdf-e9baf8707794/65afcf9b-32a3-4ef0-8354-6a9f3a5ab200"
+          (reference "U2") (unit 1)
+        )
+        (path "/994820bf-9e2d-4c1b-8cdf-e9baf8707794/5acbbc5f-2416-4b61-8e6b-a2f3458fa456"
+          (reference "U3") (unit 1)
+        )
+        (path "/994820bf-9e2d-4c1b-8cdf-e9baf8707794/eb4c094f-38d5-4c8e-a443-3cfe5211fcc9"
+          (reference "U5") (unit 1)
+        )
+      )

Commit message: More work
Parts:
- removed U1: LM5113SDE, kicad_subory:WSON10__, symbol MINI VESC-rescue:LM5001-RESCUE-MINI_VESC
- added D2: BAT46W-V, Diode_SMD:D_SOD-123, symbol Device:D_Schottky
- added R9: 100R, Resistor_SMD:R_0603_1608Metric, symbol Device:R
- U2: footprint (none) -> Footprints:WSON-10-1EP_4x4mm_P0.8mm_EP2.6x3mm_ThermalVias
Connections:
- net +5V: now also U2.1 (V_{dd}), D2.2 (A)
- net VSS: now also U2.11 (EP), U2.8 (V_{ss})
- net at Q1.1 (G), R1.1: now also U2.4 (HOL)
- net at R1.2: now also U2.3 (HOH)
- net at U2.10 (LOH): now also R6.1
- net at U2.2 (HB): now also C6.1, R9.1
- net at U2.5 (HS): now also C6.2, P1.1, Q1.2 (S), Q2.3 (D), R12.2, R7.2, R7.4, U4.8 (IN+)
- net at U2.9 (LOL): now also Q2.1 (G), R6.2
- new net: D2.1 (K), R9.2
Other:
- moved on the sheet: C2, C9, P1, P4, Q1, Q2, R1, R12, R13, R2, R6, R7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

Commit message: More work
Parts:
- removed P4: CONN_1, kicad_subory:prekov, symbol MINI VESC-rescue:CONN_1-RESCUE-MINI_VESC
- R7: value R0005 -> 500µΩ; footprint mojaKniznica:2512Rv2 -> Footprints:R_Shunt_Bourns_CSS2H-2512_6332Metric; MPN (none) -> CSS2H-2512R-L500F; Manufacturer (none) -> Bourns
Connections:
- net Phase: now reaches R7.1, R7.3, U4.1 (IN-)
Changed lines of the file:
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@@
     (stroke (width 0) (type default))
   )
-  (wire (pts (xy 207.01 77.47) (xy 209.55 77.47))
+  (wire (pts (xy 207.01 77.47) (xy 233.68 77.47))
     (stroke (width 0) (type default))
   )
@@
   (hierarchical_label "High" (shape input) (at 50.8 72.39 180) (fields_autoplaced)
     (effects (font (size 1.524 1.524)) (justify right))
+  )
+  (hierarchical_label "Phase" (shape input) (at 233.68 77.47 0) (fields_autoplaced)
+    (effects (font (size 1.524 1.524)) (justify left))
   )
   (hierarchical_label "I_{sense}" (shape input) (at 233.68 93.98 0) (fields_autoplaced)
@@
       (effects (font (size 1.27 1.27)))
     )
-    (property "Value" "R0005" (at 200.66 74.93 90)
-      (effects (font (size 1.27 1.27)))
-    )
-    (property "Footprint" "mojaKniznica:2512Rv2" (at 200.66 75.692 90)
-      (effects (font (size 1.27 1.27)) hide)
-    )
-    (property "Datasheet" "" (at 200.66 77.47 0)
-      (effects (font (size 1.27 1.27)))
+    (property "Value" "500µΩ" (at 200.66 74.93 90)
+      (effects (font (size 1.27 1.27)))
+    )
+    (property "Footprint" "Footprints:R_Shunt_Bourns_CSS2H-2512_6332Metric" (at 200.66 75.692 90)
+      (effects (font (size 1.27 1.27)) hide)
+    )
+    (property "Datasheet" "https://www.bourns.com/docs/product-datasheets/css2h-2512.pdf" (at 200.66 77.47 0)
+      (effects (font (size 1.27 1.27)) hide)
+    )
+    (property "Manufacturer" "Bourns" (at 196.215 67.945 90)
+      (effects (font (size 1.524 1.524)) (justify left))
+    )
+    (property "MPN" "CSS2H-2512R-L500F" (at 196.215 71.12 90)
+      (effects (font (size 1.524 1.524)) (justify left))
     )
     (pin "1")
@@
         )
       )
-    )
-  )
-  (symbol (lib_id "MINI VESC-rescue:CONN_1-RESCUE-MINI_VESC") (at 213.36 77.47 0) (unit 1)
-    (in_bom yes) (on_board yes) (dnp no)
-    (property "Reference" "P4" (at 215.392 77.47 0)
-      (effects (font (size 1.016 1.016)) (justify left))
-    )
-    (property "Value" "CONN_1" (at 213.36 76.073 0)
-      (effects (font (size 0.762 0.762)) hide)
-    )
-    (property "Footprint" "kicad_subory:prekov" (at 213.36 77.47 0)
-      (effects (font (size 1.524 1.524)) hide)
-    )
-    (property "Datasheet" "" (at 213.36 77.47 0)
-      (effects (font (size 1.524 1.524)))
-    )
-    (pin "1")
-    (instances
-      (project "mini-vesc"
-        (path "/994820bf-9e2d-4c1b-8cdf-e9baf8707794/65afcf9b-32a3-4ef0-8354-6a9f3a5ab200"
-          (reference "P4") (unit 1)
-        )
-        (path "/994820bf-9e2d-4c1b-8cdf-e9baf8707794/eb4c094f-38d5-4c8e-a443-3cfe5211fcc9"
-          (reference "P4") (unit 1)
-        )
-        (path "/994820bf-9e2d-4c1b-8cdf-e9baf8707794/5acbbc5f-2416-4b61-8e6b-a2f3458fa456"
-          (reference "P4") (unit 1)
-        )
-      )

Commit message: More work
Parts:
- R1, R6: value 3R9 -> 3.9Ω
- R12: value 39k -> 39kΩ
- R13: value 2k2 -> 2.2kΩ
- R2, R9: value 100R -> 100Ω
Changed lines of the file:
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@@
       (effects (font (size 1.27 1.27)))
     )
-    (property "Value" "100R" (at 220.98 96.52 90)
+    (property "Value" "100Ω" (at 220.98 96.52 90)
       (effects (font (size 1.27 1.27)))
     )
@@
       (effects (font (size 1.27 1.27)))
     )
-    (property "Value" "3R9" (at 113.03 67.31 90)
+    (property "Value" "3.9Ω" (at 113.03 67.31 90)
       (effects (font (size 1.27 1.27)))
     )
@@
       (effects (font (size 1.27 1.27)))
     )
-    (property "Value" "100R" (at 87.63 53.34 90)
+    (property "Value" "100Ω" (at 87.63 53.34 90)
       (effects (font (size 1.27 1.27)))
     )
@@
       (effects (font (size 1.27 1.27)))
     )
-    (property "Value" "39k" (at 163.83 83.82 90)
+    (property "Value" "39kΩ" (at 163.83 83.82 90)
       (effects (font (size 1.27 1.27)))
     )
@@
       (effects (font (size 1.27 1.27)))
     )
-    (property "Value" "2k2" (at 163.83 96.52 90)
+    (property "Value" "2.2kΩ" (at 163.83 96.52 90)
       (effects (font (size 1.27 1.27)))
     )
@@
       (effects (font (size 1.27 1.27)))
     )
-    (property "Value" "3R9" (at 113.03 87.63 90)
-      (effects (font (size 1.27 1.27)))
-    )
+    (property "Value" "3.9Ω" (at 113.03 87.63 90)
+      (effects (font (size 1.27 1.27)))
+    )

Commit message: Playing around with routing
Parts:
- removed D2: BAT46W-V, Diode_SMD:D_SOD-123, symbol Device:D_Schottky
- removed R9: 100Ω, Resistor_SMD:R_0603_1608Metric, symbol Device:R
- C75: renamed from C1; footprint Capacitor_SMD:C_0603_1608Metric -> Capacitor_SMD:C_0402_1005Metric
- C76: renamed from C6; footprint Capacitor_SMD:C_0603_1608Metric -> Capacitor_SMD:C_0402_1005Metric
- C77: renamed from C9; footprint Capacitor_SMD:C_0603_1608Metric -> Capacitor_SMD:C_0402_1005Metric
- C78: renamed from C2; footprint Capacitor_SMD:C_0603_1608Metric -> Capacitor_SMD:C_0402_1005Metric
- Q1, Q2: footprint kicad_subory:DFN5 -> Package_SO:ONSemi_SO-8FL_488AA; symbol Device:Q_NMOS_GSD -> Symbols:Q_NMOS_SSSGD; Manufacturer (none) -> ON Semiconductor
- R15: renamed from R1; footprint Resistor_SMD:R_0603_1608Metric -> Resistor_SMD:R_0402_1005Metric
- R16: renamed from R6; footprint Resistor_SMD:R_0603_1608Metric -> Resistor_SMD:R_0402_1005Metric
- R17: renamed from R12; footprint Resistor_SMD:R_0603_1608Metric -> Resistor_SMD:R_0402_1005Metric
- R18: renamed from R13; footprint Resistor_SMD:R_0603_1608Metric -> Resistor_SMD:R_0402_1005Metric
- R20: renamed from R2; footprint Resistor_SMD:R_0603_1608Metric -> Resistor_SMD:R_0402_1005Metric
- U3: renamed from U2; value ~ -> LM5113-Q1
- renumbered P1 to P4, R7 to R19
Connections:
- net VDD: now also Q1.5 (D); no longer Q1.3 (D)
- net VSS: now also Q2.1 (S), Q2.3 (S)
- net HighGate: now reaches R15.1, U3.4 (HOL)
- net HighGate: now also Q1.4 (G); no longer Q1.1 (G)
- net Output: now reaches C76.2, P4.1, Q1.2 (S), R17.2, R19.2, R19.4, U3.5 (HS), U4.8 (IN+)
- net Output: now also Q1.1 (S), Q1.3 (S), Q2.5 (D); no longer Q2.3 (D)
- net LowGate: now reaches R16.2, U3.9 (LOL)
- net LowGate: now also Q2.4 (G); no longer Q2.1 (G)

Commit message: Did something I think?
Parts:
- removed U3: LM5113-Q1, Footprints:WSON-10-1EP_4x4mm_P0.8mm_EP2.6x3mm_ThermalVias, symbol Symbols:LM5113-Q1
- added U3: LMG1205, Footprints:Texas_YFX0012_DSBGA-12_1.76x1.91mm_Layout3x4_P0.4mm, symbol Symbols:LMG1205
Connections:
- net +5V: now also U3.A3 (V_{dd}), U3.C4 (V_{dd})
- net High: now also U3.B4 (HI)
- net HighGate: now also U3.D1 (HOL)
- net Low: now also U3.A4 (LI)
- net LowGate: now also U3.A1 (LOL)
- net VSS: now also U3.A2 (V_{ss})
- net at R15.2: now also U3.D2 (HOH)
- net at R16.1: now also U3.B1 (LOH)
- net at C76.1: now also U3.D3 (HB)
- net Output renamed HS
- net HS: now also U3.C1 (HS), U3.D4 (HS)
Changed lines of the file:
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@@
   (junction (at 140.97 77.47) (diameter 0) (color 0 0 0 0)
   )
-  (junction (at 68.58 92.71) (diameter 0) (color 0 0 0 0)
-  )
   (junction (at 166.37 90.17) (diameter 0) (color 0 0 0 0)
   )
@@
     (stroke (width 0) (type default))
   )
-  (wire (pts (xy 66.04 90.17) (xy 66.04 92.71))
-    (stroke (width 0) (type default))
-  )
   (wire (pts (xy 196.85 83.82) (xy 196.85 81.28))
     (stroke (width 0) (type default))
@@
     (stroke (width 0) (type default))
   )
+  (wire (pts (xy 207.01 81.28) (xy 207.01 77.47))
+    (stroke (width 0) (type default))
+  )
+  (wire (pts (xy 229.87 93.98) (xy 224.79 93.98))
+    (stroke (width 0) (type default))
+  )
+  (wire (pts (xy 55.88 77.47) (xy 58.42 77.47))
+    (stroke (width 0) (type default))
+  )
+  (wire (pts (xy 68.58 52.07) (xy 68.58 55.88))
+    (stroke (width 0) (type default))
+  )
+  (wire (pts (xy 166.37 100.33) (xy 166.37 102.87))
+    (stroke (width 0) (type default))
+  )
+  (wire (pts (xy 104.14 64.77) (xy 106.68 64.77))
+    (stroke (width 0) (type default))
+  )
+  (wire (pts (xy 55.88 72.39) (xy 58.42 72.39))
+    (stroke (width 0) (type default))
+  )
+  (wire (pts (xy 78.74 82.55) (xy 119.38 82.55))
+    (stroke (width 0) (type default))
+  )
   (wire (pts (xy 68.58 90.17) (xy 68.58 92.71))
     (stroke (width 0) (type default))
   )
-  (wire (pts (xy 207.01 81.28) (xy 207.01 77.47))
-    (stroke (width 0) (type default))
-  )
-  (wire (pts (xy 229.87 93.98) (xy 224.79 93.98))
-    (stroke (width 0) (type default))
-  )
-  (wire (pts (xy 50.8 77.47) (xy 58.42 77.47))
-    (stroke (width 0) (type default))
-  )
-  (wire (pts (xy 68.58 52.07) (xy 68.58 55.88))
-    (stroke (width 0) (type default))
-  )
-  (wire (pts (xy 166.37 100.33) (xy 166.37 102.87))
-    (stroke (width 0) (type default))
-  )
-  (wire (pts (xy 104.14 64.77) (xy 106.68 64.77))
-    (stroke (width 0) (type default))
-  )
-  (wire (pts (xy 50.8 72.39) (xy 58.42 72.39))
-    (stroke (width 0) (type default))
-  )
-  (wire (pts (xy 78.74 82.55) (xy 119.38 82.55))
-    (stroke (width 0) (type default))
-  )
-  (wire (pts (xy 68.58 92.71) (xy 68.58 95.25))
-    (stroke (width 0) (type default))
-  )
   (wire (pts (xy 213.36 96.52) (xy 210.82 96.52))
     (stroke (width 0) (type default))
@@
   )
   (wire (pts (xy 229.87 93.98) (xy 229.87 97.79))
-    (stroke (width 0) (type default))
-  )
-  (wire (pts (xy 66.04 92.71) (xy 68.58 92.71))
     (stroke (width 0) (type default))
   )
@@
     (effects (font (size 1.524 1.524)) (justify left))
   )
-  (hierarchical_label "Low" (shape input) (at 50.8 77.47 180) (fields_autoplaced)
+  (hierarchical_label "Low" (shape input) (at 55.88 77.47 180) (fields_autoplaced)
     (effects (font (size 1.524 1.524)) (justify right))
   )
-  (hierarchical_label "High" (shape input) (at 50.8 72.39 180) (fields_autoplaced)
+  (hierarchical_label "High" (shape input) (at 55.88 72.39 180) (fields_autoplaced)
     (effects (font (size 1.524 1.524)) (justify right))
   )
@@
         (path "/994820bf-9e2d-4c1b-8cdf-e9baf8707794/eb4c094f-38d5-4c8e-a443-3cfe5211fcc9"
           (reference "#PWR075") (unit 1)
-        )
-      )
-    )
-  )
-  (symbol (lib_id "Symbols:LM5113-Q1") (at 68.58 74.93 0) (unit 1)
-    (in_bom yes) (on_board yes) (dnp no)
-    (property "Reference" "U3" (at 60.96 60.96 0)
-      (effects (font (size 1.27 1.27)) (justify left))
-    )
-    (property "Value" "LM5113-Q1" (at 76.2 88.9 0)
-      (effects (font (size 1.27 1.27)))
-    )
-    (property "Footprint" "Footprints:WSON-10-1EP_4x4mm_P0.8mm_EP2.6x3mm_ThermalVias" (at 68.58 73.66 0)
-      (effects (font (size 1.27 1.27)) hide)
-    )
-    (property "Datasheet" "https://www.ti.com/lit/ds/symlink/lm5113-q1.pdf" (at 68.58 73.66 0)
-      (effects (font (size 1.27 1.27)) hide)
-    )
-    (pin "8")
-    (pin "7")
-    (pin "6")
-    (pin "4")
-    (pin "9")
-    (pin "5")
-    (pin "3")
-    (pin "2")
-    (pin "11")
-    (pin "1")
-    (pin "10")
-    (instances
-      (project "mini-vesc"
-        (path "/994820bf-9e2d-4c1b-8cdf-e9baf8707794/65afcf9b-32a3-4ef0-8354-6a9f3a5ab200"
-          (reference "U3") (unit 1)
-        )
-        (path "/994820bf-9e2d-4c1b-8cdf-e9baf8707794/5acbbc5f-2416-4b61-8e6b-a2f3458fa456"
-          (reference "U5") (unit 1)
-        )
-        (path "/994820bf-9e2d-4c1b-8cdf-e9baf8707794/eb4c094f-38d5-4c8e-a443-3cfe5211fcc9"
-          (reference "U7") (unit 1)
         )
       )
@@
     )
   )
+  (symbol (lib_id "Symbols:LMG1205") (at 68.58 74.93 0) (unit 1)
+    (in_bom yes) (on_board yes) (dnp no) (fields_autoplaced)
+    (property "Reference" "U3" (at 70.7741 57.15 0)
+      (effects (font (size 1.27 1.27)) (justify left))
+    )
+    (property "Value" "LMG1205" (at 70.7741 59.69 0)
+      (effects (font (size 1.27 1.27)) (justify left))
+    )
+    (property "Footprint" "Footprints:Texas_YFX0012_DSBGA-12_1.76x1.91mm_Layout3x4_P0.4mm" (at 68.58 73.66 0)
+      (effects (font (size 1.27 1.27)) hide)
+    )
+    (property "Datasheet" "https://www.ti.com/lit/ds/symlink/lmg1205.pdf" (at 68.58 73.66 0)
+      (effects (font (size 1.27 1.27)) hide)
+    )
+    (pin "B4")
+    (pin "B1")
+    (pin "D4")
+    (pin "D2")
+    (pin "D3")
+    (pin "A2")
+    (pin "A3")
+    (pin "D1")
+    (pin "A4")
+    (pin "A1")
+    (pin "C1")
+    (pin "C4")
+    (instances
+      (project "mini-vesc"
+        (path "/994820bf-9e2d-4c1b-8cdf-e9baf8707794/65afcf9b-32a3-4ef0-8354-6a9f3a5ab200"
+          (reference "U3") (unit 1)
+        )
+        (path "/994820bf-9e2d-4c1b-8cdf-e9baf8707794/5acbbc5f-2416-4b61-8e6b-a2f3458fa456"
+          (reference "U5") (unit 1)
+        )
+        (path "/994820bf-9e2d-4c1b-8cdf-e9baf8707794/eb4c094f-38d5-4c8e-a443-3cfe5211fcc9"
+          (reference "U7") (unit 1)
+        )
+      )
+    )
+  )
   (symbol (lib_id "power:VSS") (at 140.97 92.71 180) (unit 1)
     (in_bom yes) (on_board yes) (dnp no)
@@
     )
   )
-  (symbol (lib_id "power:VSS") (at 68.58 95.25 180) (unit 1)
-    (in_bom yes) (on_board yes) (dnp no)
-    (property "Reference" "#PWR056" (at 68.58 91.44 0)
-      (effects (font (size 1.27 1.27)) hide)
-    )
-    (property "Value" "VSS" (at 68.58 99.06 0)
-      (effects (font (size 1.27 1.27)))
-    )
-    (property "Footprint" "" (at 68.58 95.25 0)
-      (effects (font (size 1.27 1.27)) hide)
-    )
-    (property "Datasheet" "" (at 68.58 95.25 0)
-      (effects (font (size 1.27 1.27)) hide)
-    )
+  (symbol (lib_id "power:VSS") (at 68.58 92.71 180) (unit 1)
+    (in_bom yes) (on_board yes) (dnp no)
+    (property "Reference" "#PWR056" (at 68.58 88.9 0)
+      (effects (font (size 1.27 1.27)) hide)
+    )
+    (property "Value" "VSS" (at 68.58 96.52 0)
+      (effects (font (size 1.27 1.27)))
+    )
+    (property "Footprint" "" (at 68.58 92.71 0)
+      (effects (font (size 1.27 1.27)) hide)
+    )
+    (property "Datasheet" "" (at 68.58 92.71 0)
+      (effects (font (size 1.27 1.27)) hide)
+    )
